Commit message: Working sim. Added changed spawn entity in gazebo ros.

File: src/vehicle_simulator/urdf/lidar.urdf.xacro (robot description, xacro)
@@ -2,5 +2,5 @@
   <link name="lidar" />
   <xacro:include filename="$(find velodyne_description)/urdf/VLP-16.urdf.xacro"/>
-  <xacro:VLP-16 parent="lidar" name="velodyne" topic="/velodyne_points" hz="5" samples="350" min_range="0.1" organize_cloud="true">
+  <xacro:VLP-16 parent="lidar" name="velodyne" topic="/velodyne_points" hz="5" samples="350" min_range="0.1">
     <origin xyz="0 0 0" rpy="0 0 0" />
   </xacro:VLP-16>

File: src/velodyne_simulator/velodyne_description/urdf/HDL-32E.urdf.xacro (robot description, xacro)
@@ -2,5 +2,5 @@
 <robot xmlns:xacro="http://www.ros.org/wiki/xacro" name="HDL-32E">
   <xacro:property name="M_PI" value="3.1415926535897931" />
-  <xacro:macro name="HDL-32E" params="*origin parent:=base_link name:=velodyne tf_prefix:='' topic:=/velodyne_points organize_cloud:=false hz:=10 lasers:=32 samples:=2187 collision_range:=0.3 min_range:=0.9 max_range:=130.0 noise:=0.008 min_angle:=-${M_PI} max_angle:=${M_PI} gpu:=false">
+  <xacro:macro name="HDL-32E" params="*origin parent:=base_link name:=velodyne topic:=/velodyne_points hz:=10 lasers:=32 samples:=2187 collision_range:=0.3 min_range:=0.9 max_range:=130.0 noise:=0.008 min_angle:=-${M_PI} max_angle:=${M_PI} gpu:=false">
     <joint name="${name}_base_mount_joint" type="fixed">
       <xacro:insert_block name="origin" />
@@ -80,14 +80,9 @@
           </ray>
           <plugin name="gazebo_ros_laser_controller" filename="libgazebo_ros_velodyne_laser.so">
-            <ros>
-              <namespace>/${name}</namespace>
-              <remapping>~/out:=${topic}</remapping>
-            </ros>
-            <tf_prefix>${tf_prefix}</tf_prefix>
-            <frame_name>${name}</frame_name>
-            <organize_cloud>${organize_cloud}</organize_cloud>
+            <topicName>${topic}</topicName>
+            <frameName>${name}</frameName>
             <min_range>${min_range}</min_range>
             <max_range>${max_range}</max_range>
-            <gaussian_noise>${noise}</gaussian_noise>
+            <gaussianNoise>${noise}</gaussianNoise>
           </plugin>
         </sensor>
@@ -125,14 +120,9 @@
           </ray>
           <plugin name="gazebo_ros_laser_controller" filename="libgazebo_ros_velodyne_laser.so">
-            <ros>
-              <namespace>/${name}</namespace>
-              <remapping>~/out:=${topic}</remapping>
-            </ros>
-            <tf_prefix>${tf_prefix}</tf_prefix>
-            <frame_name>${name}</frame_name>
-            <organize_cloud>${organize_cloud}</organize_cloud>
+            <topicName>${topic}</topicName>
+            <frameName>${name}</frameName>
             <min_range>${min_range}</min_range>
             <max_range>${max_range}</max_range>
-            <gaussian_noise>${noise}</gaussian_noise>
+            <gaussianNoise>${noise}</gaussianNoise>
           </plugin>
         </sensor>

File: src/velodyne_simulator/velodyne_description/urdf/VLP-16.urdf.xacro (robot description, xacro)
@@ -1,8 +1,8 @@
 <?xml version="1.0"?>
 <robot xmlns:xacro="http://www.ros.org/wiki/xacro" name="VLP-16">
-  <xacro:property name="M_PI" value="3.1415926535897931" />
-  <xacro:macro name="VLP-16" params="*origin parent:=base_link name:=velodyne tf_prefix:='' topic:=/velodyne_points organize_cloud:=false hz:=10 lasers:=16 samples:=1875 collision_range:=0.3 min_range:=0.9 max_range:=130.0 noise:=0.008 min_angle:=-${M_PI} max_angle:=${M_PI} gpu:=false">
+  <xacro:property name="M_PI" value="3.1415926535897931"/>
+  <xacro:macro name="VLP-16" params="*origin parent:=base_link name:=velodyne topic:=/velodyne_points hz:=10 lasers:=16 samples:=1875 collision_range:=0.3 min_range:=0.9 max_range:=130.0 noise:=0.008 min_angle:=-${M_PI} max_angle:=${M_PI} gpu:=false">
     <joint name="${name}_base_mount_joint" type="fixed">
-      <xacro:insert_block name="origin" />
+      <xacro:insert_block name="origin"/>
       <parent link="${parent}"/>
       <child link="${name}_base_link"/>
@@ -12,16 +12,14 @@
         <mass value="0.83"/>
         <origin xyz="0 0 0.03585"/>
-        <inertia ixx="${(0.83 * (3.0*0.0516*0.0516 + 0.0717*0.0717)) / 12.0}" ixy="0" ixz="0"
-          iyy="${(0.83 * (3.0*0.0516*0.0516 + 0.0717*0.0717)) / 12.0}" iyz="0"
-          izz="${0.5 * 0.83 * (0.0516*0.0516)}"/>
+        <inertia ixx="${(0.83 * (3.0*0.0516*0.0516 + 0.0717*0.0717)) / 12.0}" ixy="0" ixz="0" iyy="${(0.83 * (3.0*0.0516*0.0516 + 0.0717*0.0717)) / 12.0}" iyz="0" izz="${0.5 * 0.83 * (0.0516*0.0516)}"/>
       </inertial>
       <visual>
         <geometry>
-          <mesh filename="package://velodyne_description/meshes/VLP16_base_1.dae" />
+          <mesh filename="package://velodyne_description/meshes/VLP16_base_1.dae"/>
         </geometry>
       </visual>
       <visual>
         <geometry>
-          <mesh filename="package://velodyne_description/meshes/VLP16_base_2.dae" />
+          <mesh filename="package://velodyne_description/meshes/VLP16_base_2.dae"/>
         </geometry>
       </visual>
@@ -33,7 +31,7 @@
       </collision>
     </link>
-    <joint name="${name}_base_scan_joint" type="fixed" >
-      <origin xyz="0 0 0.0377" rpy="0 0 0" />
-      <parent link="${name}_base_link" />
+    <joint name="${name}_base_scan_joint" type="fixed">
+      <origin xyz="0 0 0.0377" rpy="0 0 0"/>
+      <parent link="${name}_base_link"/>
       <child link="${name}"/>
     </joint>
@@ -45,7 +43,7 @@
       </inertial>
       <visual>
-        <origin xyz="0 0 -0.0377" />
+        <origin xyz="0 0 -0.0377"/>
         <geometry>
-          <mesh filename="package://velodyne_description/meshes/VLP16_scan.dae" />
+          <mesh filename="package://velodyne_description/meshes/VLP16_scan.dae"/>
         </geometry>
       </visual>
@@ -70,5 +68,6 @@
                 <resolution>1</resolution>
                 <min_angle>-${15.0*M_PI/180.0}</min_angle>
-                <max_angle> ${15.0*M_PI/180.0}</max_angle>
+                <max_angle>
+                  ${15.0*M_PI/180.0}</max_angle>
               </vertical>
             </scan>
@@ -85,14 +84,9 @@
           </ray>
           <plugin name="gazebo_ros_laser_controller" filename="libgazebo_ros_velodyne_laser.so">
-            <ros>
-              <namespace>/${name}</namespace>
-              <remapping>~/out:=${topic}</remapping>
-            </ros>
-            <tf_prefix>${tf_prefix}</tf_prefix>
-            <frame_name>${name}</frame_name>
-            <organize_cloud>${organize_cloud}</organize_cloud>
+            <topicName>${topic}</topicName>
+            <frameName>${name}</frameName>
             <min_range>${min_range}</min_range>
             <max_range>${max_range}</max_range>
-            <gaussian_noise>${noise}</gaussian_noise>
+            <gaussianNoise>${noise}</gaussianNoise>
           </plugin>
         </sensor>
@@ -115,5 +109,6 @@
                 <resolution>1</resolution>
                 <min_angle>-${15.0*M_PI/180.0}</min_angle>
-                <max_angle> ${15.0*M_PI/180.0}</max_angle>
+                <max_angle>
+                  ${15.0*M_PI/180.0}</max_angle>
               </vertical>
             </scan>
@@ -130,14 +125,9 @@
           </ray>
           <plugin name="gazebo_ros_laser_controller" filename="libgazebo_ros_velodyne_laser.so">
-            <ros>
-              <namespace>/${name}</namespace>
-              <remapping>~/out:=${topic}</remapping>
-            </ros>
-            <tf_prefix>${tf_prefix}</tf_prefix>
-            <frame_name>${name}</frame_name>
-            <organize_cloud>${organize_cloud}</organize_cloud>
+            <topicName>${topic}</topicName>
+            <frameName>${name}</frameName>
             <min_range>${min_range}</min_range>
             <max_range>${max_range}</max_range>
-            <gaussian_noise>${noise}</gaussian_noise>
+            <gaussianNoise>${noise}</gaussianNoise>
           </plugin>
         </sensor>

File: src/velodyne_simulator/velodyne_description/urdf/example.urdf.xacro (robot description, xacro)
@@ -3,6 +3,4 @@
   <xacro:arg name="gpu" default="false"/>
   <xacro:property name="gpu" value="$(arg gpu)" />
-  <xacro:arg name="organize_cloud" default="false"/>
-  <xacro:property name="organize_cloud" value="$(arg organize_cloud)" />
   <!-- Base Footprint -->
   <link name="base_footprint" />
@@ -33,10 +31,14 @@
   </link>
   <xacro:include filename="$(find velodyne_description)/urdf/VLP-16.urdf.xacro"/>
-  <xacro:VLP-16 parent="base_link" name="velodyne" topic="/velodyne_points" organize_cloud="${organize_cloud}" hz="10" samples="440" gpu="${gpu}">
+  <VLP-16 parent="base_link" name="velodyne" topic="/velodyne_points" hz="10" samples="440" gpu="${gpu}">
     <origin xyz="0 0 0.4" rpy="0 0 0" />
-  </xacro:VLP-16>
+  </VLP-16>
   <xacro:include filename="$(find velodyne_description)/urdf/HDL-32E.urdf.xacro"/>
-  <xacro:HDL-32E parent="base_link" name="velodyne2" topic="/velodyne_points2" organize_cloud="${organize_cloud}" hz="10" samples="220" gpu="${gpu}">
+   <HDL-32E parent="base_link" name="velodyne2" topic="/velodyne_points2" hz="10" samples="220" gpu="${gpu}">
     <origin xyz="0 0 0.6" rpy="0 0 0" />
-  </xacro:HDL-32E>
+  </HDL-32E>
+  <xacro:include filename="$(find velodyne_description)/urdf/VLP-32C.urdf.xacro"/>
+  <VLP-32C parent="base_link" name="velodyne3" topic="/velodyne_points3" hz="10" samples="1200" gpu="${gpu}">
+    <origin xyz="0 0 0.8" rpy="0 0 0" />
+  </VLP-32C>
 </robot>

Commit message: delete gazebo_ros and modify velodyne_simulator

File: src/vehicle_simulator/urdf/lidar.urdf.xacro (robot description, xacro)
@@ -1,2 +1,3 @@
+<?xml version="1.0"?>
 <robot xmlns:xacro="http://www.ros.org/wiki/xacro" name="example">
   <link name="lidar" />

File: src/velodyne_simulator/velodyne_description/urdf/HDL-32E.urdf.xacro (robot description, xacro)
@@ -2,5 +2,5 @@
 <robot xmlns:xacro="http://www.ros.org/wiki/xacro" name="HDL-32E">
   <xacro:property name="M_PI" value="3.1415926535897931" />
-  <xacro:macro name="HDL-32E" params="*origin parent:=base_link name:=velodyne topic:=/velodyne_points hz:=10 lasers:=32 samples:=2187 collision_range:=0.3 min_range:=0.9 max_range:=130.0 noise:=0.008 min_angle:=-${M_PI} max_angle:=${M_PI} gpu:=false">
+  <xacro:macro name="HDL-32E" params="*origin parent:=base_link name:=velodyne tf_prefix:='' topic:=/velodyne_points organize_cloud:=false hz:=10 lasers:=32 samples:=2187 collision_range:=0.3 min_range:=0.9 max_range:=130.0 noise:=0.008 min_angle:=-${M_PI} max_angle:=${M_PI} gpu:=false">
     <joint name="${name}_base_mount_joint" type="fixed">
       <xacro:insert_block name="origin" />
@@ -80,9 +80,14 @@
           </ray>
           <plugin name="gazebo_ros_laser_controller" filename="libgazebo_ros_velodyne_laser.so">
-            <topicName>${topic}</topicName>
-            <frameName>${name}</frameName>
+            <ros>
+              <namespace>/${name}</namespace>
+              <remapping>~/out:=${topic}</remapping>
+            </ros>
+            <tf_prefix>${tf_prefix}</tf_prefix>
+            <frame_name>${name}</frame_name>
+            <organize_cloud>${organize_cloud}</organize_cloud>
             <min_range>${min_range}</min_range>
             <max_range>${max_range}</max_range>
-            <gaussianNoise>${noise}</gaussianNoise>
+            <gaussian_noise>${noise}</gaussian_noise>
           </plugin>
         </sensor>
@@ -120,9 +125,14 @@
           </ray>
           <plugin name="gazebo_ros_laser_controller" filename="libgazebo_ros_velodyne_laser.so">
-            <topicName>${topic}</topicName>
-            <frameName>${name}</frameName>
+            <ros>
+              <namespace>/${name}</namespace>
+              <remapping>~/out:=${topic}</remapping>
+            </ros>
+            <tf_prefix>${tf_prefix}</tf_prefix>
+            <frame_name>${name}</frame_name>
+            <organize_cloud>${organize_cloud}</organize_cloud>
             <min_range>${min_range}</min_range>
             <max_range>${max_range}</max_range>
-            <gaussianNoise>${noise}</gaussianNoise>
+            <gaussian_noise>${noise}</gaussian_noise>
           </plugin>
         </sensor>

File: src/velodyne_simulator/velodyne_description/urdf/VLP-16.urdf.xacro (robot description, xacro)
@@ -1,8 +1,8 @@
 <?xml version="1.0"?>
 <robot xmlns:xacro="http://www.ros.org/wiki/xacro" name="VLP-16">
-  <xacro:property name="M_PI" value="3.1415926535897931"/>
-  <xacro:macro name="VLP-16" params="*origin parent:=base_link name:=velodyne topic:=/velodyne_points hz:=10 lasers:=16 samples:=1875 collision_range:=0.3 min_range:=0.9 max_range:=130.0 noise:=0.008 min_angle:=-${M_PI} max_angle:=${M_PI} gpu:=false">
+  <xacro:property name="M_PI" value="3.1415926535897931" />
+  <xacro:macro name="VLP-16" params="*origin parent:=base_link name:=velodyne tf_prefix:='' topic:=/velodyne_points organize_cloud:=false hz:=10 lasers:=16 samples:=1875 collision_range:=0.3 min_range:=0.9 max_range:=130.0 noise:=0.008 min_angle:=-${M_PI} max_angle:=${M_PI} gpu:=false">
     <joint name="${name}_base_mount_joint" type="fixed">
-      <xacro:insert_block name="origin"/>
+      <xacro:insert_block name="origin" />
       <parent link="${parent}"/>
       <child link="${name}_base_link"/>
@@ -12,14 +12,16 @@
         <mass value="0.83"/>
         <origin xyz="0 0 0.03585"/>
-        <inertia ixx="${(0.83 * (3.0*0.0516*0.0516 + 0.0717*0.0717)) / 12.0}" ixy="0" ixz="0" iyy="${(0.83 * (3.0*0.0516*0.0516 + 0.0717*0.0717)) / 12.0}" iyz="0" izz="${0.5 * 0.83 * (0.0516*0.0516)}"/>
+        <inertia ixx="${(0.83 * (3.0*0.0516*0.0516 + 0.0717*0.0717)) / 12.0}" ixy="0" ixz="0"
+          iyy="${(0.83 * (3.0*0.0516*0.0516 + 0.0717*0.0717)) / 12.0}" iyz="0"
+          izz="${0.5 * 0.83 * (0.0516*0.0516)}"/>
       </inertial>
       <visual>
         <geometry>
-          <mesh filename="package://velodyne_description/meshes/VLP16_base_1.dae"/>
+          <mesh filename="package://velodyne_description/meshes/VLP16_base_1.dae" />
         </geometry>
       </visual>
       <visual>
         <geometry>
-          <mesh filename="package://velodyne_description/meshes/VLP16_base_2.dae"/>
+          <mesh filename="package://velodyne_description/meshes/VLP16_base_2.dae" />
         </geometry>
       </visual>
@@ -31,7 +33,7 @@
       </collision>
     </link>
-    <joint name="${name}_base_scan_joint" type="fixed">
-      <origin xyz="0 0 0.0377" rpy="0 0 0"/>
-      <parent link="${name}_base_link"/>
+    <joint name="${name}_base_scan_joint" type="fixed" >
+      <origin xyz="0 0 0.0377" rpy="0 0 0" />
+      <parent link="${name}_base_link" />
       <child link="${name}"/>
     </joint>
@@ -43,7 +45,7 @@
       </inertial>
       <visual>
-        <origin xyz="0 0 -0.0377"/>
+        <origin xyz="0 0 -0.0377" />
         <geometry>
-          <mesh filename="package://velodyne_description/meshes/VLP16_scan.dae"/>
+          <mesh filename="package://velodyne_description/meshes/VLP16_scan.dae" />
         </geometry>
       </visual>
@@ -68,6 +70,5 @@
                 <resolution>1</resolution>
                 <min_angle>-${15.0*M_PI/180.0}</min_angle>
-                <max_angle>
-                  ${15.0*M_PI/180.0}</max_angle>
+                <max_angle> ${15.0*M_PI/180.0}</max_angle>
               </vertical>
             </scan>
@@ -84,9 +85,14 @@
           </ray>
           <plugin name="gazebo_ros_laser_controller" filename="libgazebo_ros_velodyne_laser.so">
-            <topicName>${topic}</topicName>
-            <frameName>${name}</frameName>
+            <ros>
+              <namespace>/${name}</namespace>
+              <remapping>~/out:=${topic}</remapping>
+            </ros>
+            <tf_prefix>${tf_prefix}</tf_prefix>
+            <frame_name>${name}</frame_name>
+            <organize_cloud>${organize_cloud}</organize_cloud>
             <min_range>${min_range}</min_range>
             <max_range>${max_range}</max_range>
-            <gaussianNoise>${noise}</gaussianNoise>
+            <gaussian_noise>${noise}</gaussian_noise>
           </plugin>
         </sensor>
@@ -109,6 +115,5 @@
                 <resolution>1</resolution>
                 <min_angle>-${15.0*M_PI/180.0}</min_angle>
-                <max_angle>
-                  ${15.0*M_PI/180.0}</max_angle>
+                <max_angle> ${15.0*M_PI/180.0}</max_angle>
               </vertical>
             </scan>
@@ -125,9 +130,14 @@
           </ray>
           <plugin name="gazebo_ros_laser_controller" filename="libgazebo_ros_velodyne_laser.so">
-            <topicName>${topic}</topicName>
-            <frameName>${name}</frameName>
+            <ros>
+              <namespace>/${name}</namespace>
+              <remapping>~/out:=${topic}</remapping>
+            </ros>
+            <tf_prefix>${tf_prefix}</tf_prefix>
+            <frame_name>${name}</frame_name>
+            <organize_cloud>${organize_cloud}</organize_cloud>
             <min_range>${min_range}</min_range>
             <max_range>${max_range}</max_range>
-            <gaussianNoise>${noise}</gaussianNoise>
+            <gaussian_noise>${noise}</gaussian_noise>
           </plugin>
         </sensor>

File: src/velodyne_simulator/velodyne_description/urdf/example.urdf.xacro (robot description, xacro)
@@ -3,4 +3,6 @@
   <xacro:arg name="gpu" default="false"/>
   <xacro:property name="gpu" value="$(arg gpu)" />
+  <xacro:arg name="organize_cloud" default="false"/>
+  <xacro:property name="organize_cloud" value="$(arg organize_cloud)" />
   <!-- Base Footprint -->
   <link name="base_footprint" />
@@ -31,14 +33,10 @@
   </link>
   <xacro:include filename="$(find velodyne_description)/urdf/VLP-16.urdf.xacro"/>
-  <VLP-16 parent="base_link" name="velodyne" topic="/velodyne_points" hz="10" samples="440" gpu="${gpu}">
+  <xacro:VLP-16 parent="base_link" name="velodyne" topic="/velodyne_points" organize_cloud="${organize_cloud}" hz="10" samples="440" gpu="${gpu}">
     <origin xyz="0 0 0.4" rpy="0 0 0" />
-  </VLP-16>
+  </xacro:VLP-16>
   <xacro:include filename="$(find velodyne_description)/urdf/HDL-32E.urdf.xacro"/>
-   <HDL-32E parent="base_link" name="velodyne2" topic="/velodyne_points2" hz="10" samples="220" gpu="${gpu}">
+  <xacro:HDL-32E parent="base_link" name="velodyne2" topic="/velodyne_points2" organize_cloud="${organize_cloud}" hz="10" samples="220" gpu="${gpu}">
     <origin xyz="0 0 0.6" rpy="0 0 0" />
-  </HDL-32E>
-  <xacro:include filename="$(find velodyne_description)/urdf/VLP-32C.urdf.xacro"/>
-  <VLP-32C parent="base_link" name="velodyne3" topic="/velodyne_points3" hz="10" samples="1200" gpu="${gpu}">
-    <origin xyz="0 0 0.8" rpy="0 0 0" />
-  </VLP-32C>
+  </xacro:HDL-32E>
 </robot>
