Commit message: add gmapping

File: src/vehicle_simulator/urdf/robot.urdf.xacro (robot description, xacro)
@@ -1,3 +1,4 @@
 <robot xmlns:xacro="http://www.ros.org/wiki/xacro" name="example">
+  <xacro:include filename="$(find vehicle_simulator)/urdf/hokuyo.gazebo" />
   <xacro:macro name="gazebo_material" params="ref color">
     <gazebo reference="${ref}">
@@ -118,4 +119,29 @@
     <child link="right_rear_wheel"/>
   </joint>
+  <link name="hokuyo">
+    <collision>
+      <origin xyz="0 0 0" rpy="0 0 0"/>
+      <geometry>
+        <box size="0.1 0.1 0.1"/>
+      </geometry>
+    </collision>
+    <visual>
+      <origin xyz="0 0 0" rpy="0 0 0"/>
+      <geometry>
+        <mesh filename="package://vehicle_simulator/meshes/hokuyo.dae"/>
+      </geometry>
+    </visual>
+    <inertial>
+      <mass value="1e-5" />
+      <origin xyz="0 0 0" rpy="0 0 0"/>
+      <inertia ixx="1e-6" ixy="0" ixz="0" iyy="1e-6" iyz="0" izz="1e-6" />
+    </inertial>
+  </link>
+  <joint name="hokuyo_joint" type="fixed">
+    <axis xyz="0 1 0" />
+    <origin xyz=".0 0 .4" rpy="0 0 0"/>
+    <parent link="base_link"/>
+    <child link="hokuyo"/>
+  </joint>
   <xacro:gazebo_material ref="base_link"         color="Red" />
   <xacro:gazebo_material ref="lidar_holder"      color="Black" />
